File: BMS.kicad_sch (KiCad schematic)
At the start: 48 parts, among them J1 BATT+, J2 LOAD, J3 BATT-, J4 QWIIC, J5 PROG, Q1 SI2333, Q2 SI2333, Q3 SI2333, U1 TLV61070ADBV, U2 ATtiny824-SSU

Commit message: Finished schematic
Parts:
- C1, C2, C3, C7: footprint (none) -> Capacitor_SMD:C_0402_1005Metric_Pad0.74x0.62mm_HandSolder
- C4, C5, C6: footprint (none) -> Capacitor_SMD:C_0603_1608Metric_Pad1.08x0.95mm_HandSolder
- F1, F2: footprint (none) -> Fuse:Fuse_0805_2012Metric_Pad1.15x1.40mm_HandSolder
- J1, J3: footprint (none) -> MountingHole:MountingHole_3.2mm_M3_ISO7380_Pad_TopOnly
- J2: footprint (none) -> TerminalBlock_RND:TerminalBlock_RND_205-00012_1x02_P5.00mm_Horizontal
- J4: footprint (none) -> Connector_PinHeader_2.54mm:PinHeader_1x04_P2.54mm_Horizontal; symbol Connector_Generic_MountingPin:Conn_01x04_MountingPin -> Connector_Generic:Conn_01x04
- J5: footprint (none) -> Connector_PinHeader_2.54mm:PinHeader_1x03_P2.54mm_Vertical
- JP1, JP2: footprint (none) -> Jumper:SolderJumper-2_P1.3mm_Open_RoundedPad1.0x1.5mm
- L1: footprint (none) -> Inductor_SMD:L_1812_4532Metric_Pad1.30x3.40mm_HandSolder
- Q1, Q2, Q3: footprint Package_TO_SOT_SMD:SOT-23-3 -> Package_TO_SOT_SMD:SOT-23
- R1, R14: footprint (none) -> Resistor_SMD:R_1206_3216Metric_Pad1.30x1.75mm_HandSolder
- R10, R11, R12, R13, R15, R16, R2, R3, R4, R5, R6, R7, R8, R9: footprint (none) -> Resistor_SMD:R_0402_1005Metric_Pad0.72x0.64mm_HandSolder
- TP1, TP10, TP2, TP3, TP4, TP5, TP6, TP7, TP8, TP9: footprint (none) -> TestPoint:TestPoint_Pad_1.0x1.0mm; now left out of the parts list
Connections:
- net GND: no longer J4.MP (MountPin)

Commit message: First PCB design
Parts:
- renumbered R12 to R10, R15 to R12, R9 to R14, R14 to R15, R13 to R16, R10 to R17, R16 to R9
Connections:
- net ADC_SP: now also J4.2 (Pin_2); no longer J4.1 (Pin_1)
- net SCL: now also R10.2; no longer R11.2
- net SDA: now also R11.2; no longer R10.2
- net at R11.1, TP7.1: now also J4.3 (Pin_3); no longer J4.4 (Pin_4)
- net at R10.1, TP8.1: now also J4.4 (Pin_4); no longer J4.3 (Pin_3)
- net at JP2.1 (A): now also J4.1 (Pin_1); no longer J4.2 (Pin_2)
Other:
- moved on the sheet: F2, JP2, Q3, R10, R11, R15, R16, TP10, TP7, TP8
